File: uhome.sch (KiCad schematic (older format))
At the start: 31 parts, among them J1 C2, J2 ANT, U1 Si7006, U2 LPS22HB, U3 EFM8SB10, U4 Si4012, U5 AH1806

Commit message: Revision 2
Parts:
- removed C2: 0.1µ, Capacitors_SMD:C_0402_NoSilk, symbol C
- removed R3: 600, Resistors_SMD:R_0402_NoSilk, symbol R
- removed R4: 13k, Resistors_SMD:R_0402_NoSilk, symbol R
- removed R5: 11k, Resistors_SMD:R_0402_NoSilk, symbol R
- removed U2: LPS22HB, ufqfn:HLGA-10L, symbol LPS22HB
- added C5, C7: 4.5pF, Capacitors_SMD:C_0402_NoSilk, symbol C
- added J2, J4: Conn_01x02, Buttons_Switches_SMD:SW_SPST_B3U-1000P, symbol Conn_01x02
- added J3: Conn_01x04, Pin_Headers:Pin_Header_Straight_2x02_Pitch2.00mm_SMD, symbol Conn_01x04
- added L1, L2: 30nH, Capacitors_SMD:C_0402_NoSilk, symbol L
- C10: renamed from C9; value CM5 -> CM5 (6.8pF)
- C11: renamed from C10; value CM1 -> CM1 (4.3pF)
- C12: renamed from C11; value CM2 -> CM2 (1.8 pF)
- C13: renamed from C12; value CM3 -> CM3 (2.7pF)
- C6: value CC1 -> 15pF
- C9: renamed from C8; value CM6 -> CM6 (6.8pF)
- L3: renamed from L1; value LM5 -> LM5 (18nH)
- L4: renamed from L2; value LM3 -> LM3 (56 nH)
- L5: renamed from L3; value LM2 -> LM2 (16 nH)
- L6: renamed from L4; value LM4 -> LM4 (16 nH)
- L7: renamed from L5; value LM1 -> LM1 (220 nH)
- renumbered C3 to C1, C4 to C2, C1 to C3, C5 to C4, C7 to C8, J2 to J5, U3 to U2, U5 to U3
Connections:
- net GND: now also C6.2, C5.2, C7.2, J2.2 (Pin_2), J4.1 (Pin_1)
- net at U2.10 (P1.3): now also J4.2 (Pin_2)
- net at U2.18 (P0.4): now also J3.3 (Pin_3)
- net at U2.19 (P0.3): now also J3.2 (Pin_2)
- net at U2.20 (P0.2): now also J3.1 (Pin_1)
- net at U2.7 (P1.7): now also J2.1 (Pin_1)
- net at C9.1, L3.2: now also C7.1, L2.1; no longer C6.1
- net at J5.1 (P1): now also C5.1, L1.2; no longer C6.2
- net LPS_IRQ: no longer names the net of U2.17 (P0.5)
- net LPS_IRQ: now also J3.4 (Pin_4)
- new net: C6.1, L1.1, L2.2
Other:
- moved on the sheet: BT1, C1, C2, C4, C8, D1, J1, J5, U2, U3, U4
